File: hardware/KnGXT.kicad_sch (KiCad schematic)
At the start: 134 parts, among them J1 USB_C_ReceptacleUSB2.0, J2 Conn_01x10_Male, SW1 RotaryEncoder_Switch, SW10 SW_Push, SW11 SW_Push, SW12 SW_Push, SW13 SW_Push, SW14 SW_Push, SW15 SW_Push, SW16 SW_Push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

Commit message: Update version, date, and license in schematic
Signed-off-by: Flynn <flynn+github@kodachi.com>
Other:
- company: © 2022 kodachi 6•14, llc -> © 2022 kodachi 6•14, llc // SPDX-License-Identifier: CERN-OHL-S-2.0
Changed lines of the file:
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@@
   (title_block
     (title "KnGXT MacroPaw")
-    (date "2022-05-10")
-    (rev "v1")
-    (company "© 2022 kodachi 6•14, llc")
-    (comment 1 "https://github.com/tjhorner/bizcard")
-    (comment 2 "and TJ Horner's RP2040 business card")
+    (date "2022-08-13")
+    (rev "v0.1.0")
+    (company "© 2022 kodachi 6•14, llc // SPDX-License-Identifier: CERN-OHL-S-2.0")
+    (comment 1 "Open Source Hardware, CERN OHL 2.0: https://ohwr.org/cern_ohl_s_v2.txt")
+    (comment 2 "and TJ Horner's RP2040 business card https://github.com/tjhorner/bizcard")
     (comment 3 "https://datasheets.raspberrypi.com/rp2040/hardware-design-with-rp2040.pdf")
-    (comment 4 "Largely based off \"Hardware Design with RP2040\"")
+    (comment 4 "With grateful thanks to \"Hardware Design with RP2040\"")
   )
   (junction (at 277.114 75.946) (diameter 0) (color 0 0 0 0)
