File: KnGXT/hardware/KnGXT.kicad_pcb (KiCad board)
At the start: 2 copper layers, 94 x 108.3 mm, 136 parts, among them J1 USB_C_ReceptacleUSB2.0, J2 Conn_01x10_Male, SW1 RotaryEncoder_Switch, SW10 SW_Push, SW11 SW_Push, SW12 SW_Push, SW13 SW_Push, SW14 SW_Push, SW15 SW_Push, SW16 SW_Push, SW17 SW_Push, SW2 RotaryEncoder_Switch, SW3 SW_Push, SW4 SW_Push, SW5 SW_Push, SW6 SW_Push, SW7 SW_Push, SW8 SW_Push, SW9 SW_Push, U1 AMS1117-3.3, U2 W25Q128JVS, U3 RP2040, U4 74125, Y1 12MHz

Commit message: (Mostly?) update KnGXT for KiCad 7 and to use kicadlib.
KnGXT probably still needs work to pass ERC & DRC, but that's OK because any new spin of it will make further changes.
Parts:
- NP0, NP10, NP11, NP12, NP13, NP14, NP15, NP16, NP17, NP18, NP19, NP2, NP20, NP21, NP22, NP23, NP24, NP25, NP26, NP27, NP28, NP29, NP3, NP4, NP5, NP6, NP7, NP8, NP9: footprint LED_SMD:LED_WS2812B_3.5x2.8_C2890364 -> Kodachi:LED XL-3528RGBW-WS2812B (3.5x2.8, C2890364)
- U3: footprint RP_Silicon:RP2040-QFN-56 -> MCU_RaspberryPi_and_Boards:RP2040-QFN-56
- locked: renamed from NP1; footprint LED_SMD:LED_WS2812B_3.5x2.8_C2890364 -> Kodachi:LED XL-3528RGBW-WS2812B (3.5x2.8, C2890364)
- turned NP0 to -20 degrees
- turned NP10 to -60 degrees
- turned NP11 to -80 degrees
- turned NP12 to -100 degrees
- turned NP13 to -120 degrees
- turned NP14 to -140 degrees
- turned NP15 to -160 degrees
- turned NP16 to 180 degrees
- turned NP17 to 180 degrees
- turned NP18 to 180 degrees
- turned NP19 to 180 degrees
- turned NP2 to -60 degrees
- turned NP20 to 180 degrees
- turned NP21 to 180 degrees
- turned NP22 to 180 degrees
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